File: hw/pi3_hat.sch (EAGLE design)
At the start: 36 parts, among them U1 MAX13431E, U2 RT829910L_DFN, U3 STM32F051X6UFQFPN32, U4 DMMT5401, U5 DMG2305UX, X1 8.0MHz

Commit message: Beginnings of r4 with multiple FD-CAN busses
Parts:
- removed JD1: JST-XH4SMT_RA, odroid_shield:JST-XH4SMT_RA
- removed SWD: JST-ZH6SMT_VERT, controller:JST-ZH6SMT_VERT
- removed U1: MAX13431E, controller:MAX13431E
- removed U3: STM32F051X6UFQFPN32, pi3_hat:STM32F051X6UFQFPN32
- removed X1: 8.0MHz, controller:CRYSTALABM3B
- added C14, C16: .1uF 50V, mfpassives:CAPACITOR_NP_0805
- added C15: 0.01uF, mfpassives:CAPACITOR_NP_0603
- added C17: 3.3nF, mfpassives:CAPACITOR_NP_0402
- added C18, C19, C20, C22, C23, C24, C25, C27, C28, C29, C31, C32, C33, C34, C36, C38, C39: 0.1uF, mfpassives:CAPACITOR_NP_0402
- added C21, C30, C37: 10uF, mfpassives:CAPACITOR_NP_1206
- added C26, C35: 1uF, mfpassives:CAPACITOR_NP_0402
- added D3, D4, D5, D6: MF-LED-0603-RED, mfleds:LED_SINGLE-0603-RED
- added IC1, IC2, IC3: STM32G474CEU6, pi3_hat:STM32G474CEU6
- added JP2: (no value), pinhead:PINHD-2X20
- added R11: 14k, mfpassives:RESISTOR_0402
- added R12: 115k, mfpassives:RESISTOR_0402
- added R13: 22.1k, mfpassives:RESISTOR_0402
- added R15: 120, mfpassives:RESISTOR_0402
- added R16, R17: (no value), mfpassives:RESISTOR_0402
- added U$1, U$7: XT30P, pi3_hat:XT30P
- added U$10, U$11, U$16, U$4, U$5: JST-PH3SMT_VERT, pi3_hat:JST-PH3SMT_VERT
- added U$12, U$17, U$6: JST-ZH6SMT_VERT, pi3_hat:JST-ZH6SMT_VERT
- added U$14, U$2, U$3, U$8, U$9: TCAN334GSOT23, pi3_hat:TCAN334GSOT23
- added U$18: BMI088LGA16, pi3_hat:BMI088LGA16
- C1, C3: value .1uF 50V -> 0.1uF; device mfpassives:CAPACITOR_NP_0805 -> mfpassives:CAPACITOR_NP_0402; HOUSEPART 1 -> YES; MPN MF-CAP-0805-0.1uF -> MF-CAP-0402-0.1uF
- C10: value 10pF -> 10uF; device mfpassives:CAPACITOR_NP_0603 -> mfpassives:CAPACITOR_NP_1206; HOUSEPART 1 -> YES; MF MACROFAB -> (none); MPN MF-CAP-0603-10pF -> MF-CAP-1206-10uF
- C11: value .1uF 50V -> 1uF; device mfpassives:CAPACITOR_NP_0805 -> mfpassives:CAPACITOR_NP_0402; HOUSEPART 1 -> YES; MPN MF-CAP-0805-0.1uF -> MF-CAP-0402-1uF
- C12: value .1uF 50V -> 10uF; device mfpassives:CAPACITOR_NP_0805 -> mfpassives:CAPACITOR_NP_1206; HOUSEPART 1 -> YES; MPN MF-CAP-0805-0.1uF -> MF-CAP-1206-10uF
- C13, C4, C7: value 1uF -> 0.1uF; device mfpassives:CAPACITOR_NP_0603 -> mfpassives:CAPACITOR_NP_0402; HOUSEPART 1 -> YES; MPN MF-CAP-0603-1uF -> MF-CAP-0402-0.1uF
- C2, C6: value 10uF 35V -> 10uF 50V; MPN CGA5L1X7R1V106K160AC -> CGA5L1X7R1H106K160AC
- C9: value 10pF -> 0.1uF; device mfpassives:CAPACITOR_NP_0603 -> mfpassives:CAPACITOR_NP_0402; HOUSEPART 1 -> YES; MF MACROFAB -> (none); MPN MF-CAP-0603-10pF -> MF-CAP-0402-0.1uF
- D2: value MF-LED-0603-GREEN -> MF-LED-0603-RED; device mfleds:LED_SINGLE-0603-GREEN -> mfleds:LED_SINGLE-0603-RED
- JP1: device pinhead:PINHD-2X8 -> pinhead:PINHD-2X4; POPULATE 0 -> (none)
- R1: value 53.6k 1% -> 120; device mfpassives:RESISTOR_0603 -> mfpassives:RESISTOR_0402; MF Panasonic -> (none); MPN ERJ-3EKF5362V -> (none)
- R10: value 53.6k 1% -> (none); device mfpassives:RESISTOR_0603 -> mfpassives:RESISTOR_0402; MF Panasonic -> (none); MPN ERJ-3EKF5362V -> (none)
- R2: value 10k 1% -> 120; device mfpassives:RESISTOR_0603 -> mfpassives:RESISTOR_0402; MF Panasonic -> (none); MPN ERJ-3EKF1002V -> (none)
- R5, R6, R9: value 220 -> (none); device mfpassives:RESISTOR_0603 -> mfpassives:RESISTOR_0402; MPN MF-RES-0603-220 -> (none)
- R7, R8: value 220 -> 120; device mfpassives:RESISTOR_0603 -> mfpassives:RESISTOR_0402; MPN MF-RES-0603-220 -> (none)
- U2: value RT829910L_DFN -> AP64351SO8EP; device pi3_hat:RT829910L_DFN -> pi3_hat:AP64351SO8EP; POPULATE 1 -> (none)
Connections:
- removed net +18V: F1.1, JD1.4
- removed net 485_DIR: U1.DE, U1.RE/, U3.PA1/USART2_RTS/TIM2_CH2/ADC1
- removed net 485_RX: U1.RO, U3.PA3/USART2_RX/TIM2_CH4/TIM15_CH2
- removed net 485_TX: U1.DI, U3.PA2/USART2_TX/TIM2_CH3/TIM15_CH1/ADC2
- removed net NRST: C11.P$1, SWD.2, U3.NRST
- removed net PI_RX_3V: JP1.10, U3.PA9/USART1_TX/TIM1_CH2
- removed net POSTFUSE: C2.P$1, C6.P$1, F1.2, R10.P$1, U2.VIN
- removed net RS485_N: JD1.2, R6.P$1, R9.P$1, U1.B
- removed net RS485_P: JD1.3, R6.P$2, R9.P$2, U1.A
- removed net SW: C3.P$2, L1.P$1, U2.SW
- new net I2C1_SCL: JP2.5
- new net I2C1_SDA: JP2.3
- new net ID_SCL: JP2.28
- new net ID_SDA: JP2.27
- new net IMU_ACC_INT: IC3.PA8, U$18.INT1
- new net IMU_CS1: IC3.PB12, U$18.CSB1
- new net IMU_CS2: IC3.PB11, U$18.CSB2
- new net IMU_GYRO_INT: IC3.PA9, U$18.INT3
- new net IMU_MISO: IC3.PB14, U$18.SDO1, U$18.SDO2
- new net IMU_MOSI: IC3.PB15, U$18.SDI
- new net IMU_SCK: IC3.PB13, U$18.SCK
- new net N$10: C14.P$1, C2.P$1, C6.P$1, F1.2, U2.EN, U2.VIN
- new net N$14: C16.P$1, U2.BST
- new net N$19: C15.P$1, U2.SS
- new net N$20: C16.P$2, L1.P$1, U2.SW
- new net N$21: C17.P$1, R11.P$2
- new net N$22: R11.P$1, U2.COMP
- new net N$23: R7.P$1, U$10.1, U$8.CANH
- new net N$24: R12.P$2, R13.P$1, U2.FB
- new net N$25: R7.P$2, U$10.2, U$8.CANL
- new net N$26: R8.P$1, U$11.1, U$9.CANH
- new net N$27: R8.P$2, U$11.2, U$9.CANL
- new net N$28: D1.ANODE, R5.P$2
- new net N$29: D1.CATHODE, IC1.PC14-OSC32_IN
- new net N$30: D2.ANODE, R6.P$2
- new net N$31: D2.CATHODE, IC1.PC15-OSC32_OUT
- new net N$32: C20.P$1, IC2.PG10-NRST, U$12.2
- new net N$33: IC2.PA13, U$12.3
- new net N$34: IC2.PA14, U$12.5
- new net N$37: D4.ANODE, R10.P$2
- new net N$38: D4.CATHODE, IC2.PC15-OSC32_OUT
- new net N$39: IC2.PA11, U$9.RXD
- new net N$40: IC2.PA12, U$9.TXD
- new net N$41: IC2.PB5, U$8.RXD
- new net N$42: IC2.PB6, U$8.TXD
- new net N$45: R15.P$1, U$14.CANH, U$16.1
- new net N$46: R15.P$2, U$14.CANL, U$16.2
- new net N$47: C29.P$1, IC3.PG10-NRST, U$17.2
- new net N$48: IC3.PA13, U$17.3
- new net N$49: IC3.PA14, U$17.5
- new net N$50: D5.ANODE, R16.P$2
- new net N$51: D5.CATHODE, IC3.PC14-OSC32_IN
- new net N$52: D6.ANODE, R17.P$2
- new net N$53: D6.CATHODE, IC3.PC15-OSC32_OUT
- new net N$54: IC3.PA11, U$14.RXD
- new net N$55: IC3.PA12, U$14.TXD
- new net N$9: F1.1, U$1.2, U$7.2
- new net NRF_CE: IC3.PA15, JP1.6
- new net NRF_CS: IC3.PB6, JP1.5
- new net NRF_IRQ: IC3.PB7, JP1.1
- new net NRF_MISO: IC3.PB4, JP1.2
- new net NRF_MOSI: IC3.PB5, JP1.3
- new net NRF_SCK: IC3.PB3, JP1.4
- new net SPI0_CS0: IC3.PA4, JP2.24
- new net SPI0_CS1: JP2.26
- new net SPI0_MISO: IC3.PA6, JP2.21
- new net SPI0_MOSI: IC3.PA7, JP2.19
- new net SPI0_SCLK: IC3.PA5, JP2.23
- new net SPI1_CS0: IC1.PA4, JP2.12
- new net SPI1_CS1: IC2.PA4, JP2.11
- new net SPI1_CS2: JP2.36
- new net SPI1_MISO: IC1.PA6, IC2.PA6, JP2.35
- new net SPI1_MOSI: IC1.PA7, IC2.PA7, JP2.38
- new net SPI1_SCLK: IC1.PA5, IC2.PA5, JP2.40
- net +3V3: now also C10.P$1, C11.P$1, C18.P$1, C19.P$1, C21.P$1, C22.P$1, C23.P$1, C24.P$1, C25.P$1, C26.P$1, C27.P$1, C28.P$1, C3.P$1, C30.P$1, C31.P$1, C32.P$1, C33.P$1, C34.P$1, C35.P$1, C36.P$1, C37.P$1, C38.P$1, C39.P$1, C7.P$1, C9.P$1, IC1.VDDA, IC1.VDD_1, IC1.VDD_2, IC1.VDD_3, IC1.VREF+, IC2.VDDA, IC2.VDD_1, IC2.VDD_2, IC2.VDD_3, IC2.VREF+, IC3.VDDA, IC3.VDD_1, IC3.VDD_2, IC3.VDD_3, IC3.VREF+, JP1.7, JP2.1, JP2.17, R10.P$1, R16.P$1, R17.P$1, R5.P$1, R6.P$1, R9.P$1, U$12.6, U$14.VCC, U$17.6, U$18.VDD, U$18.VDDIO, U$2.VCC, U$3.VCC, U$6.6, U$8.VCC, U$9.VCC; no longer C1.P$1, JP1.1, R7.P$2, R8.P$2, SWD.6, U1.VCC, U1.VL, U3.VDD, U3.VDDA
- net +5V: now also JP2.2, JP2.4; no longer JP1.2, JP1.4
- net GND: now also C14.P$2, C15.P$2, C17.P$2, C18.P$2, C19.P$2, C20.P$2, C21.P$2, C22.P$2, C23.P$2, C24.P$2, C25.P$2, C26.P$2, C27.P$2, C28.P$2, C29.P$2, C3.P$2, C30.P$2, C31.P$2, C32.P$2, C33.P$2, C34.P$2, C35.P$2, C36.P$2, C37.P$2, C38.P$2, C39.P$2, IC1.THERMALPAD, IC1.VSSA, IC1.VSS_1, IC1.VSS_2, IC1.VSS_3, IC2.THERMALPAD, IC2.VSSA, IC2.VSS_1, IC2.VSS_2, IC2.VSS_3, IC3.THERMALPAD, IC3.VSSA, IC3.VSS_1, IC3.VSS_2, IC3.VSS_3, JP1.8, JP2.14, JP2.20, JP2.25, JP2.30, JP2.34, JP2.39, JP2.6, JP2.9, R13.P$2, U$1.1, U$10.3, U$11.3, U$12.4, U$14.GND, U$14.SHDN, U$14.STB, U$16.3, U$17.4, U$18.GND, U$18.GNDIO, U$18.PS, U$2.GND, U$2.SHDN, U$2.STB, U$3.GND, U$3.SHDN, U$3.STB, U$4.3, U$5.3, U$6.4, U$7.1, U$8.GND, U$8.SHDN, U$8.STB, U$9.GND, U$9.SHDN, U$9.STB; no longer JD1.1, JP1.14, JP1.6, JP1.9, R2.P$2, R5.P$2, SWD.4, U1.GND, U3.VSS, X1.P$3
- net N$11: now also IC1.PA11, U$3.RXD; no longer R1.P$2, R2.P$1, U2.FB
- net N$12: now also IC1.PA12, U$3.TXD; no longer SWD.5, U3.PA14/SWCLK
- net N$13: now also C1.P$1, IC1.PG10-NRST, U$6.2; no longer SWD.3, U3.PA13/SWDIO
- net N$15: now also IC1.PA13, U$6.3; no longer D1.ANODE, R7.P$1
- net N$16: now also IC1.PA14, U$6.5; no longer D2.ANODE, R8.P$1
- net N$17: now also IC1.PB5, U$2.RXD; no longer D1.CATHODE, U3.PB3/SPI1_SCK/TIM2_CH2
- net N$18: now also IC1.PB6, U$2.TXD; no longer D2.CATHODE, U3.PB4/SPI1_MISO/TIM3_CH1
- net N$2: now also R1.P$1, U$2.CANH, U$4.1; no longer C7.P$1, U2.VCC
- net N$35: now also D3.ANODE, R9.P$2; no longer C9.P$1, U3.PF1-OSC_OUT, X1.P$1
- net N$36: now also D3.CATHODE, IC2.PC14-OSC32_IN; no longer C10.P$1, U3.PF0-OSC_IN, X1.P$2
- net N$4: now also R1.P$2, U$2.CANL, U$4.2; no longer R5.P$1, U3.BOOT0
- net N$7: now also R2.P$1, U$3.CANH, U$5.1; no longer R10.P$2, U2.EN
- net N$8: now also R2.P$2, U$3.CANL, U$5.2; no longer C3.P$1, U2.BOOT
- net PI_TX_3V: now also JP2.8; no longer JP1.8, U3.PA10/USART1_RX/TIM1_CH3
- net REGOUT: now also R12.P$1; no longer R1.P$1
Other:
- note added: "AUX / IMU"
- note added: "IFACE A"
- note added: "IFACE B"
- note added: "INPUT POWER"
- note added: "RPI HEADER"
- note added: "mjmech pi3 hat r4 (c) jjp@pobox.com 2019 Licensed under the Apache 2.0 License"
- moved on the sheet: C1, C10, C11, C12, C13, C2, C3, C4, C5, C6, C7, C8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

Commit message: Fix up stm32 pinouts, add eeprom and test points
Parts:
- removed IC1: STM32G474CEU6, pi3_hat:STM32G474CEU6
- removed U$2: TCAN334GSOT23, pi3_hat:TCAN334GSOT23
- added +5V, GND, REGOUT, SPI0_CS0, SPI0_MISO, SPI0_MOSI, SPI0_SCLK, SPI1_CS0, SPI1_CS1, SPI1_MISO, SPI1_MOSI, SPI1_SCLK, V+: PAD24AWG_PAD, pi3_hat:PAD24AWG_PAD
- added C40: 0.1uF, mfpassives:CAPACITOR_NP_0402
- added J3: (no value), pinhead:PINHD-2X4
- added R14: 1k, mfpassives:RESISTOR_0402
- added R18, R19: 3.9k 1%, mfpassives:RESISTOR_0402
- added U1: AP64351SO8EP, pi3_hat:AP64351SO8EP
- added U10: CAT24C32SOIC8, pi3_hat:CAT24C32SOIC8
- added U3: DMG2305UX, pi3_hat:DMG2305UX
- JP1: device pinhead:PINHD-2X4 -> pinhead:PINHD-1X2
- U2: value AP64351SO8EP -> DMMT5401; device pi3_hat:AP64351SO8EP -> pi3_hat:DMMT5401; DPN (none) -> DMMT5401-FDICT-ND; MF (none) -> Didoes Incorporated; MPN (none) -> DMMT5401-7-F; POPULATE (none) -> 1
- U4: value DMMT5401 -> STM32G474CEU6; device pi3_hat:DMMT5401 -> pi3_hat:STM32G474CEU6; DPN DMMT5401-FDICT-ND -> (none); MF Didoes Incorporated -> (none); MPN DMMT5401-7-F -> (none); POPULATE 1 -> (none)
- U5: value DMG2305UX -> TCAN334GSOT23; device pi3_hat:DMG2305UX -> pi3_hat:TCAN334GSOT23; DPN DMG2305UX-13DICT-ND -> (none); MF Diodes Incorporated -> (none); MPN DMG2305UX-13 -> (none); POPULATE 1 -> (none)
- renumbered IC2 to U11, IC3 to U7, JP2 to J4, U$1 to J2, U$10 to JC4, U$11 to JC5, U$12 to JD3, U$14 to U9, U$16 to JC3, U$17 to JD2, U$18 to U8, U$3 to U6, U$4 to JC1, U$5 to JC2, U$6 to JD1, U$7 to J1, U$8 to U12, U$9 to U13
Connections:
- removed net N$12: IC1.PA12, U6.TXD
- removed net N$9: F1.1, J1.2, J2.2
- new net N$100: U4.PA12, U6.TXD
- new net N$44: JP1.2, R14.P$2, U10.WP
- new net V+: F1.1, J1.2, J2.2, V+.P$1
- net +3V3: now also C40.P$1, J3.7, R14.P$1, R18.P$1, R19.P$1, U10.VCC, U11.PC15-OSC32_OUT, U4.VBAT, U4.VDDA, U4.VDD_1, U4.VDD_2, U4.VDD_3, U4.VREF+, U5.VCC, U7.PC14-OSC32_IN; no longer IC1.VDDA, IC1.VDD_1, IC1.VDD_2, IC1.VDD_3, IC1.VREF+, JP1.7, U$2.VCC
- net +5V: now also +5V.P$1, U2.E1, U3.D; no longer U4.E1, U5.D
- net GND: now also C40.P$2, GND.P$1, J3.8, JP1.1, U1.GND, U10.A0, U10.A1, U10.A2, U10.VSS, U11.PC14-OSC32_IN, U4.PC14-OSC32_IN, U4.PC15-OSC32_OUT, U4.THERMALPAD, U5.GND, U5.SHDN, U5.STB, U7.PC15-OSC32_OUT; no longer IC1.THERMALPAD, IC1.VSSA, IC1.VSS_1, IC1.VSS_2, IC1.VSS_3, JP1.8, U$2.GND, U$2.SHDN, U$2.STB, U11.VSSA, U11.VSS_1, U11.VSS_2, U11.VSS_3, U2.GND, U7.VSSA, U7.VSS_1, U7.VSS_2, U7.VSS_3
- net ID_SCL: now also R19.P$2, U10.SCL
- net ID_SDA: now also R18.P$2, U10.SDA
- net N$1: now also U2.B1, U2.B2, U2.C2; no longer U4.B1, U4.B2, U4.C2
- net N$10: now also U1.EN, U1.VIN; no longer U2.EN, U2.VIN
- net N$11: now also U4.PA11; no longer IC1.PA11
- net N$13: now also U4.PG10-NRST; no longer IC1.PG10-NRST
- net N$14: now also U1.BST; no longer U2.BST
- net N$15: now also U4.PA13; no longer IC1.PA13
- net N$16: now also U4.PA14; no longer IC1.PA14
- net N$17: now also U4.PB3, U5.RXD; no longer IC1.PB5, U$2.RXD
- net N$18: now also U4.PB4, U5.TXD; no longer IC1.PB6, U$2.TXD
- net N$19: now also U1.SS; no longer U2.SS
- net N$2: now also U5.CANH; no longer U$2.CANH
- net N$20: now also U1.SW; no longer U2.SW
- net N$22: now also U1.COMP; no longer U2.COMP
- net N$24: now also U1.FB; no longer U2.FB
- net N$29: now also U4.PF0-OSC_IN; no longer IC1.PC14-OSC32_IN
- net N$31: now also U4.PF1-OSC_OUT; no longer IC1.PC15-OSC32_OUT
- net N$36: now also U11.PF0-OSC_IN; no longer U11.PC14-OSC32_IN
- net N$38: now also U11.PF1-OSC_OUT; no longer U11.PC15-OSC32_OUT
- net N$4: now also U5.CANL; no longer U$2.CANL
- net N$41: now also U11.PB3; no longer U11.PB5
- net N$42: now also U11.PB4; no longer U11.PB6
- net N$5: now also U2.C1, U3.G; no longer U4.C1, U5.G
- net N$51: now also U7.PF0-OSC_IN; no longer U7.PC14-OSC32_IN
- net N$53: now also U7.PF1-OSC_OUT; no longer U7.PC15-OSC32_OUT
- net NRF_CE: now also J3.6, U7.PB6; no longer JP1.6, U7.PA15
- net NRF_CS: now also J3.5, U7.PA15; no longer JP1.5, U7.PB6
- net NRF_IRQ: now also J3.1; no longer JP1.1
- net NRF_MISO: now also J3.2; no longer JP1.2
- net NRF_MOSI: now also J3.3; no longer JP1.3
- net NRF_SCK: now also J3.4; no longer JP1.4
- net REGOUT: now also REGOUT.P$1, U2.E2, U3.S; no longer U4.E2, U5.S
- net SPI0_CS0: now also SPI0_CS0.P$1
- net SPI0_MISO: now also SPI0_MISO.P$1
- net SPI0_MOSI: now also SPI0_MOSI.P$1
- net SPI0_SCLK: now also SPI0_SCLK.P$1
- net SPI1_CS0: now also SPI1_CS0.P$1, U4.PA4; no longer IC1.PA4
- net SPI1_CS1: now also SPI1_CS1.P$1
- net SPI1_MISO: now also SPI1_MISO.P$1, U4.PA6; no longer IC1.PA6
- net SPI1_MOSI: now also SPI1_MOSI.P$1, U4.PA7; no longer IC1.PA7
- net SPI1_SCLK: now also SPI1_SCLK.P$1, U4.PA5; no longer IC1.PA5
Other:
- note added: "DEVICE 0x0 (00)"
- note added: "DEVICE 0x1 (01)"
- note added: "DEVICE 0x2 (10)"
- note added: "TEST POINTS"
- note added: "mjmech pi3 hat r4 (c) jjp@pobox.com 2020 Licensed under the Apache 2.0 License"
- note removed: "mjmech pi3 hat r4 (c) jjp@pobox.com 2019 Licensed under the Apache 2.0 License"
- moved on the sheet: C1

Commit message: Rough place all components
Parts:
- removed R6: (no value), mfpassives:RESISTOR_0402
- added D7: MF-LED-0603-RED, mfleds:LED_SINGLE-0603-RED
- added D8: 36V, pi3_hat:SMF
- added F6: 53.6k 1%, mfpassives:RESISTOR_0603
- added R20: 120, mfpassives:RESISTOR_0402
- C1: value 0.1uF -> .1uF 50V; device mfpassives:CAPACITOR_NP_0402 -> mfpassives:CAPACITOR_NP_0805; HOUSEPART YES -> 1; MPN MF-CAP-0402-0.1uF -> MF-CAP-0805-0.1uF
- C10, C12, C21, C30: value 10uF -> 0.1uF; device mfpassives:CAPACITOR_NP_1206 -> mfpassives:CAPACITOR_NP_0402; MPN MF-CAP-1206-10uF -> MF-CAP-0402-0.1uF
- C14: value .1uF 50V -> 10uF; device mfpassives:CAPACITOR_NP_0805 -> mfpassives:CAPACITOR_NP_1206; HOUSEPART 1 -> YES; MPN MF-CAP-0805-0.1uF -> MF-CAP-1206-10uF
- C15: value 0.01uF -> 0.1uF; device mfpassives:CAPACITOR_NP_0603 -> mfpassives:CAPACITOR_NP_0402; HOUSEPART (none) -> YES; MPN MF-CAP-0603-0.01uF -> MF-CAP-0402-0.1uF
- C16: value .1uF 50V -> 0.1uF; device mfpassives:CAPACITOR_NP_0805 -> mfpassives:CAPACITOR_NP_0402; HOUSEPART 1 -> YES; MPN MF-CAP-0805-0.1uF -> MF-CAP-0402-0.1uF
- C17: value 3.3nF -> 0.1uF; HOUSEPART (none) -> YES; MPN (none) -> MF-CAP-0402-0.1uF
- C20, C34: value 0.1uF -> 1uF; MPN MF-CAP-0402-0.1uF -> MF-CAP-0402-1uF
- C23, C29: value 0.1uF -> 10uF; device mfpassives:CAPACITOR_NP_0402 -> mfpassives:CAPACITOR_NP_1206; MPN MF-CAP-0402-0.1uF -> MF-CAP-1206-10uF
- C26: value 1uF -> 10uF; device mfpassives:CAPACITOR_NP_0402 -> mfpassives:CAPACITOR_NP_1206; MPN MF-CAP-0402-1uF -> MF-CAP-1206-10uF
- C3: value 0.1uF -> 10uF 50V; device mfpassives:CAPACITOR_NP_0402 -> mfpassives:CAPACITOR_NP_1206; HOUSEPART YES -> (none); MF (none) -> TDK; MPN MF-CAP-0402-0.1uF -> CGA5L1X7R1H106K160AC
- C35: value 1uF -> 0.1uF; MPN MF-CAP-0402-1uF -> MF-CAP-0402-0.1uF
- C4: value 0.1uF -> 0.01uF; device mfpassives:CAPACITOR_NP_0402 -> mfpassives:CAPACITOR_NP_0603; HOUSEPART YES -> (none); MPN MF-CAP-0402-0.1uF -> MF-CAP-0603-0.01uF
- C5: value 22uF 16V -> .1uF 50V; device mfpassives:CAPACITOR_NP_1210 -> mfpassives:CAPACITOR_NP_0805; HOUSEPART (none) -> 1; MF SAMSUNG -> (none); MPN CL32A226KOJNNNE -> MF-CAP-0805-0.1uF
- C6: value 10uF 50V -> 3.3nF; device mfpassives:CAPACITOR_NP_1206 -> mfpassives:CAPACITOR_NP_0402; MF TDK -> (none); MPN CGA5L1X7R1H106K160AC -> (none)
- C7: value 0.1uF -> 22uF 16V; device mfpassives:CAPACITOR_NP_0402 -> mfpassives:CAPACITOR_NP_1210; HOUSEPART YES -> (none); MF (none) -> SAMSUNG; MPN MF-CAP-0402-0.1uF -> CL32A226KOJNNNE
- R1: value 120 -> 14k
- R10, R9: value (none) -> 120
- R11: value 14k -> 220
- R12: value 115k -> 220
- R13: value 22.1k -> 120
- R15: value 120 -> 3.9k 1%
- R16: value (none) -> 3.9k 1%
- R17: value (none) -> 220
- R18: value 3.9k 1% -> 220
- R19: value 3.9k 1% -> 120
- R2: value 120 -> 115k
- R3: value 10k 1% -> 22.1k; device mfpassives:RESISTOR_0603 -> mfpassives:RESISTOR_0402; MF Panasonic -> (none); MPN ERJ-3EKF1002V -> (none)
- R4: value 53.6k 1% -> ~700; device mfpassives:RESISTOR_0603 -> mfpassives:RESISTOR_0402; MF Panasonic -> (none); MPN ERJ-3EKF5362V -> (none)
- R5: value (none) -> 10k 1%; device mfpassives:RESISTOR_0402 -> mfpassives:RESISTOR_0603; MF (none) -> Panasonic; MPN (none) -> ERJ-3EKF1002V
- R7, R8: value 120 -> 220
Connections:
- removed net N$37 (its old number): D4.ANODE, R10.P$2
- new net N$52: D4.ANODE, R11.P$2
- new net N$9: D1.ANODE, R4.P$2
- net +3V3: now also C14.P$1, C15.P$1, C16.P$1, C17.P$1, C20.P$1, C29.P$1, R11.P$1, R12.P$1, R15.P$1, R7.P$1, R8.P$1, U11.VBAT, U7.VBAT; no longer C18.P$1, C3.P$1, C32.P$1, C4.P$1, C7.P$1, C9.P$1, R10.P$1, R19.P$1, R5.P$1, R6.P$1, R9.P$1
- net +5V: now also R4.P$1
- net GND: now also C16.P$2, D1.CATHODE, D8.A, F6.P$2, R5.P$2; no longer C5.P$2, R13.P$2, R4.P$2
- net ID_SCL: now also R16.P$2; no longer R19.P$2
- net ID_SDA: now also R15.P$2; no longer R18.P$2
- net N$1: now also R5.P$1; no longer R3.P$1
- net N$10: now also C1.P$1, C3.P$1, D8.C; no longer C14.P$1, C6.P$1
- net N$13: now also C9.P$1; no longer C1.P$1
- net N$14: now also C5.P$1; no longer C16.P$1
- net N$19: now also C4.P$1; no longer C15.P$1
- net N$2: now also R9.P$1; no longer R1.P$1
- net N$20: now also C5.P$2; no longer C16.P$2
- net N$21: now also C6.P$1, R1.P$2; no longer C17.P$1, R11.P$2
- net N$22: now also R1.P$1; no longer R11.P$1
- net N$23: now also R19.P$1; no longer R7.P$1
- net N$24: now also R2.P$2, R3.P$1; no longer R12.P$2, R13.P$1
- net N$25: now also R19.P$2; no longer R7.P$2
- net N$26: now also R20.P$1; no longer R8.P$1
- net N$27: now also R20.P$2; no longer R8.P$2
- net N$28: now also D3.ANODE, R8.P$2; no longer D1.ANODE, R5.P$2
- net N$29: now also D3.CATHODE; no longer D1.CATHODE
- net N$30: now also R7.P$2; no longer R6.P$2
- net N$32: now also C32.P$1; no longer C20.P$1
- net N$35: now also D7.ANODE, R18.P$2; no longer D3.ANODE, R9.P$2
- net N$36: now also D7.CATHODE; no longer D3.CATHODE
- net N$38: now also D6.CATHODE; no longer D4.CATHODE
- net N$4: now also R9.P$2; no longer R1.P$2
- net N$45: now also R13.P$1; no longer R15.P$1
- net N$46: now also R13.P$2; no longer R15.P$2
- net N$47: now also C18.P$1; no longer C29.P$1
- net N$5: now also F6.P$1; no longer R4.P$1
- net N$50: now also R12.P$2; no longer R16.P$2
- net N$53: now also D4.CATHODE; no longer D6.CATHODE
- net N$7: now also R10.P$1; no longer R2.P$1
- net N$8: now also R10.P$2; no longer R2.P$2
- net REGOUT: now also C7.P$1, R2.P$1; no longer C5.P$1, R12.P$1
Other:
- moved on the sheet: C1, C10, C12, C13, C14, C15, C16, C17, C18, C19, C2, C20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

Commit message: Rough silks
Connections:
- net N$23: now also JC3.1; no longer JC4.1
- net N$25: now also JC3.2; no longer JC4.2
- net N$26: now also JC4.1; no longer JC5.1
- net N$27: now also JC4.2; no longer JC5.2
- net N$45: now also JC5.1; no longer JC3.1
- net N$46: now also JC5.2; no longer JC3.2
Other:
- moved on the sheet: JC3, JC4, JC5
Changed lines of the file:
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@@
 <part name="U12" library="pi3_hat" deviceset="TCAN334G" device="SOT23"/>
 <part name="U13" library="pi3_hat" deviceset="TCAN334G" device="SOT23"/>
+<part name="JC3" library="pi3_hat" deviceset="JST-PH3" device="SMT_VERT"/>
 <part name="JC4" library="pi3_hat" deviceset="JST-PH3" device="SMT_VERT"/>
-<part name="JC5" library="pi3_hat" deviceset="JST-PH3" device="SMT_VERT"/>
 <part name="R19" library="mfpassives" deviceset="RESISTOR" device="_0402" value="120"/>
 <part name="R20" library="mfpassives" deviceset="RESISTOR" device="_0402" value="120"/>
@@
 <part name="U7" library="pi3_hat" deviceset="STM32G474CEU6" device=""/>
 <part name="U9" library="pi3_hat" deviceset="TCAN334G" device="SOT23"/>
-<part name="JC3" library="pi3_hat" deviceset="JST-PH3" device="SMT_VERT"/>
+<part name="JC5" library="pi3_hat" deviceset="JST-PH3" device="SMT_VERT"/>
 <part name="R13" library="mfpassives" deviceset="RESISTOR" device="_0402" value="120"/>
 <part name="GND38" library="supply1" deviceset="GND" device=""/>
@@
 <instance part="U12" gate="G$1" x="464.82" y="83.82"/>
 <instance part="U13" gate="G$1" x="464.82" y="45.72"/>
-<instance part="JC4" gate="A" x="541.02" y="83.82" rot="MR0"/>
-<instance part="JC5" gate="A" x="541.02" y="45.72" rot="MR0"/>
+<instance part="JC3" gate="A" x="541.02" y="83.82" rot="MR0"/>
+<instance part="JC4" gate="A" x="541.02" y="45.72" rot="MR0"/>
 <instance part="R19" gate="G$1" x="520.7" y="81.28" rot="R90"/>
 <instance part="R20" gate="G$1" x="520.7" y="43.18" rot="R90"/>
@@
 <instance part="U7" gate="G$1" x="670.56" y="251.46"/>
 <instance part="U9" gate="G$1" x="779.78" y="226.06"/>
-<instance part="JC3" gate="A" x="855.98" y="226.06" rot="MR0"/>
+<instance part="JC5" gate="A" x="855.98" y="226.06" rot="MR0"/>
 <instance part="R13" gate="G$1" x="835.66" y="223.52" rot="R90"/>
 <instance part="GND38" gate="1" x="848.36" y="210.82"/>
@@
 </segment>
 <segment>
-<pinref part="JC4" gate="A" pin="3"/>
+<pinref part="JC3" gate="A" pin="3"/>
 <pinref part="GND26" gate="1" pin="GND"/>
 <wire x1="535.94" y1="81.28" x2="533.4" y2="81.28" width="0.1524" layer="91"/>
@@
 </segment>
 <segment>
-<pinref part="JC5" gate="A" pin="3"/>
+<pinref part="JC4" gate="A" pin="3"/>
 <pinref part="GND25" gate="1" pin="GND"/>
 <wire x1="535.94" y1="43.18" x2="533.4" y2="43.18" width="0.1524" layer="91"/>
@@
 </segment>
 <segment>
-<pinref part="JC3" gate="A" pin="3"/>
+<pinref part="JC5" gate="A" pin="3"/>
 <pinref part="GND38" gate="1" pin="GND"/>
 <wire x1="850.9" y1="223.52" x2="848.36" y2="223.52" width="0.1524" layer="91"/>
@@
 <wire x1="515.62" y1="81.28" x2="515.62" y2="86.36" width="0.1524" layer="91"/>
 <junction x="515.62" y="81.28"/>
-<pinref part="JC4" gate="A" pin="1"/>
+<pinref part="JC3" gate="A" pin="1"/>
 <wire x1="515.62" y1="86.36" x2="535.94" y2="86.36" width="0.1524" layer="91"/>
 </segment>
@@
 <wire x1="525.78" y1="81.28" x2="525.78" y2="83.82" width="0.1524" layer="91"/>
 <junction x="525.78" y="81.28"/>
-<pinref part="JC4" gate="A" pin="2"/>
+<pinref part="JC3" gate="A" pin="2"/>
 <wire x1="525.78" y1="83.82" x2="535.94" y2="83.82" width="0.1524" layer="91"/>
 </segment>
@@
 <wire x1="515.62" y1="43.18" x2="515.62" y2="48.26" width="0.1524" layer="91"/>
 <junction x="515.62" y="43.18"/>
-<pinref part="JC5" gate="A" pin="1"/>
+<pinref part="JC4" gate="A" pin="1"/>
 <wire x1="515.62" y1="48.26" x2="535.94" y2="48.26" width="0.1524" layer="91"/>
 </segment>
@@
 <wire x1="525.78" y1="43.18" x2="525.78" y2="45.72" width="0.1524" layer="91"/>
 <junction x="525.78" y="43.18"/>
-<pinref part="JC5" gate="A" pin="2"/>
+<pinref part="JC4" gate="A" pin="2"/>
 <wire x1="525.78" y1="45.72" x2="535.94" y2="45.72" width="0.1524" layer="91"/>
 </segment>
@@
 <wire x1="830.58" y1="223.52" x2="830.58" y2="228.6" width="0.1524" layer="91"/>
 <junction x="830.58" y="223.52"/>
-<pinref part="JC3" gate="A" pin="1"/>
+<pinref part="JC5" gate="A" pin="1"/>
 <wire x1="830.58" y1="228.6" x2="850.9" y2="228.6" width="0.1524" layer="91"/>
 </segment>
@@
 <wire x1="840.74" y1="223.52" x2="840.74" y2="226.06" width="0.1524" layer="91"/>
 <junction x="840.74" y="223.52"/>
-<pinref part="JC3" gate="A" pin="2"/>
+<pinref part="JC5" gate="A" pin="2"/>
 <wire x1="840.74" y1="226.06" x2="850.9" y2="226.06" width="0.1524" layer="91"/>
 </segment>
