File: hw/pi3_hat.sch (EAGLE design)
At the start: 110 parts, among them J1 XT30P, J2 XT30P, U1 AP64351SO8EP, U10 CAT24C32SOIC8, U11 STM32G474CEU6, U12 TCAN334GSOT23, U13 TCAN334GSOT23, U2 DMMT5401, U3 DMG2305UX, U4 STM32G474CEU6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

Commit message: Fix R5/R6 to use parts that are the correct size
Parts:
- R5: MPN RC0402FR-0710KL -> RC0603FR-0710KL
- R6: MPN RC0402FR-0753K6L -> RC0603FR-0753K6L
Changed lines of the file:
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@@
 <part name="R5" library="mfpassives" deviceset="RESISTOR" device="_0603" value="10k 1%">
 <attribute name="MF" value="YAGEO"/>
-<attribute name="MPN" value="RC0402FR-0710KL"/>
+<attribute name="MPN" value="RC0603FR-0710KL"/>
 </part>
 <part name="R6" library="mfpassives" deviceset="RESISTOR" device="_0603" value="53.6k 1%">
 <attribute name="MF" value="YAGEO"/>
-<attribute name="MPN" value="RC0402FR-0753K6L"/>
+<attribute name="MPN" value="RC0603FR-0753K6L"/>
 </part>
 <part name="J2" library="pi3_hat" deviceset="XT30" device="P">

Commit message: Basic SPI slave operation that works at least a little
Parts:
- U1: MPN (none) -> AP64351SP-13
Other:
- note added: "mjbots quad pi3 hat r4.1 (c) jjp@pobox.com 2020 Licensed under the Apache 2.0 License"
- note removed: "mjbots quad pi3 hat r4 (c) jjp@pobox.com 2020 Licensed under the Apache 2.0 License"
Changed lines of the file:
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@@
 </part>
 <part name="GND11" library="supply1" deviceset="GND" device=""/>
-<part name="U1" library="pi3_hat" deviceset="AP64351" device="SO8EP"/>
+<part name="U1" library="pi3_hat" deviceset="AP64351" device="SO8EP">
+<attribute name="MPN" value="AP64351SP-13"/>
+</part>
 <part name="GND12" library="supply1" deviceset="GND" device=""/>
 <part name="C4" library="mfpassives" deviceset="CAPACITOR_NP" device="_0603" value="0.01uF">
@@
 <wire x1="-48.26" y1="170.18" x2="-48.26" y2="347.98" width="0.1524" layer="90"/>
 <text x="-45.72" y="335.28" size="7.62" layer="90" font="vector">INPUT POWER</text>
-<text x="-45.72" y="355.6" size="7.62" layer="90" font="vector">mjbots quad pi3 hat r4
+<text x="-45.72" y="355.6" size="7.62" layer="90" font="vector">mjbots quad pi3 hat r4.1
 (c) jjp@pobox.com 2020
 Licensed under the Apache 2.0 License</text>

Commit message: Add mjbots logo
Other:
- note added: "mjbots pi3 hat r4.2 (c) jjp@pobox.com 2020 Licensed under the Apache 2.0 License"
- note removed: "mjbots quad pi3 hat r4.1 (c) jjp@pobox.com 2020 Licensed under the Apache 2.0 License"
Changed lines of the file:
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@@
 <wire x1="-48.26" y1="170.18" x2="-48.26" y2="347.98" width="0.1524" layer="90"/>
 <text x="-45.72" y="335.28" size="7.62" layer="90" font="vector">INPUT POWER</text>
-<text x="-45.72" y="355.6" size="7.62" layer="90" font="vector">mjbots quad pi3 hat r4.1
+<text x="-45.72" y="355.6" size="7.62" layer="90" font="vector">mjbots pi3 hat r4.2
 (c) jjp@pobox.com 2020
 Licensed under the Apache 2.0 License</text>

Commit message: Add debug pads for each processor
Parts:
- added DBG1A, DBG1B, DBG2A, DBG2B, DBG3A, DBG3B: PAD24AWG_PAD, pi3_hat:PAD24AWG_PAD
Connections:
- new net DBG1A: DBG1A.P$1, U4.PB13
- new net DBG1B: DBG1B.P$1, U4.PB12
- new net DBG2A: DBG2A.P$1, U11.PB13
- new net DBG2B: DBG2B.P$1, U11.PB12
- new net DBG3A: DBG3A.P$1, U7.PA2
- new net DBG3B: DBG3B.P$1, U7.PA3
Changed lines of the file:
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@@
+<attribute name="POPULATE" value="0"/>
+</part>
+<part name="DBG1A" library="pi3_hat" deviceset="PAD" device="24AWG_PAD">
+<attribute name="POPULATE" value="0"/>
+</part>
+<part name="DBG1B" library="pi3_hat" deviceset="PAD" device="24AWG_PAD">
+<attribute name="POPULATE" value="0"/>
+</part>
+<part name="DBG2A" library="pi3_hat" deviceset="PAD" device="24AWG_PAD">
+<attribute name="POPULATE" value="0"/>
+</part>
+<part name="DBG2B" library="pi3_hat" deviceset="PAD" device="24AWG_PAD">
+<attribute name="POPULATE" value="0"/>
+</part>
+<part name="DBG3A" library="pi3_hat" deviceset="PAD" device="24AWG_PAD">
+<attribute name="POPULATE" value="0"/>
+</part>
+<part name="DBG3B" library="pi3_hat" deviceset="PAD" device="24AWG_PAD">
 <attribute name="POPULATE" value="0"/>
 </part>
@@
 <instance part="GND54" gate="1" x="347.98" y="50.8"/>
 <instance part="+3V29" gate="G$1" x="345.44" y="73.66"/>
-<instance part="GND55" gate="1" x="662.94" y="231.14"/>
+<instance part="GND55" gate="1" x="657.86" y="231.14"/>
 <instance part="+3V30" gate="G$1" x="657.86" y="254"/>
 <instance part="REGOUT" gate="G$1" x="728.98" y="134.62">
@@
 <instance part="3V3_TP" gate="G$1" x="728.98" y="66.04">
 <attribute name="POPULATE" x="728.98" y="66.04" size="1.778" layer="96" display="off"/>
+</instance>
+<instance part="DBG1A" gate="G$1" x="787.4" y="137.16">
+<attribute name="POPULATE" x="787.4" y="137.16" size="1.778" layer="96" display="off"/>
+</instance>
+<instance part="DBG1B" gate="G$1" x="787.4" y="124.46">
+<attribute name="POPULATE" x="787.4" y="124.46" size="1.778" layer="96" display="off"/>
+</instance>
+<instance part="DBG2A" gate="G$1" x="787.4" y="101.6">
+<attribute name="POPULATE" x="787.4" y="101.6" size="1.778" layer="96" display="off"/>
+</instance>
+<instance part="DBG2B" gate="G$1" x="787.4" y="88.9">
+<attribute name="POPULATE" x="787.4" y="88.9" size="1.778" layer="96" display="off"/>
+</instance>
+<instance part="DBG3A" gate="G$1" x="787.4" y="71.12">
+<attribute name="POPULATE" x="787.4" y="71.12" size="1.778" layer="96" display="off"/>
+</instance>
+<instance part="DBG3B" gate="G$1" x="787.4" y="58.42">
+<attribute name="POPULATE" x="787.4" y="58.42" size="1.778" layer="96" display="off"/>
 </instance>
 </instances>
@@
 <segment>
 <pinref part="GND55" gate="1" pin="GND"/>
-<wire x1="662.94" y1="233.68" x2="662.94" y2="243.84" width="0.1524" layer="91"/>
+<wire x1="657.86" y1="233.68" x2="662.94" y2="243.84" width="0.1524" layer="91"/>
 <pinref part="U7" gate="G$1" pin="PC15-OSC32_OUT"/>
 <wire x1="662.94" y1="243.84" x2="670.56" y2="243.84" width="0.1524" layer="91"/>
@@
 </segment>
 </net>
+<net name="DBG1A" class="0">
+<segment>
+<pinref part="DBG1A" gate="G$1" pin="P$1"/>
+<wire x1="779.78" y1="137.16" x2="767.08" y2="137.16" width="0.1524" layer="91"/>
+<label x="767.08" y="137.16" size="1.778" layer="95"/>
+</segment>
+<segment>
+<pinref part="U4" gate="G$1" pin="PB13"/>
+<wire x1="403.86" y1="226.06" x2="419.1" y2="226.06" width="0.1524" layer="91"/>
+<label x="414.02" y="226.06" size="1.778" layer="95"/>
+</segment>
+</net>
+<net name="DBG1B" class="0">
+<segment>
+<pinref part="DBG1B" gate="G$1" pin="P$1"/>
+<wire x1="779.78" y1="124.46" x2="767.08" y2="124.46" width="0.1524" layer="91"/>
+<label x="767.08" y="124.46" size="1.778" layer="95"/>
+</segment>
+<segment>
+<pinref part="U4" gate="G$1" pin="PB12"/>
+<wire x1="403.86" y1="223.52" x2="419.1" y2="223.52" width="0.1524" layer="91"/>
+<label x="414.02" y="223.52" size="1.778" layer="95"/>
+</segment>
+</net>
+<net name="DBG2A" class="0">
+<segment>
+<pinref part="DBG2A" gate="G$1" pin="P$1"/>
+<wire x1="779.78" y1="101.6" x2="767.08" y2="101.6" width="0.1524" layer="91"/>
+<label x="767.08" y="101.6" size="1.778" layer="95"/>
+</segment>
+<segment>
+<pinref part="U11" gate="G$1" pin="PB13"/>
+<wire x1="401.32" y1="45.72" x2="416.56" y2="45.72" width="0.1524" layer="91"/>
+<label x="411.48" y="45.72" size="1.778" layer="95"/>
+</segment>
+</net>
+<net name="DBG2B" class="0">
+<segment>
+<pinref part="DBG2B" gate="G$1" pin="P$1"/>
+<wire x1="779.78" y1="88.9" x2="767.08" y2="88.9" width="0.1524" layer="91"/>
+<label x="767.08" y="88.9" size="1.778" layer="95"/>
+</segment>
+<segment>
+<pinref part="U11" gate="G$1" pin="PB12"/>
+<wire x1="401.32" y1="43.18" x2="416.56" y2="43.18" width="0.1524" layer="91"/>
+<label x="411.48" y="43.18" size="1.778" layer="95"/>
+</segment>
+</net>
+<net name="DBG3A" class="0">
+<segment>
+<pinref part="DBG3A" gate="G$1" pin="P$1"/>
+<wire x1="779.78" y1="71.12" x2="767.08" y2="71.12" width="0.1524" layer="91"/>
+<label x="767.08" y="71.12" size="1.778" layer="95"/>
+</segment>
+<segment>
+<pinref part="U7" gate="G$1" pin="PA2"/>
+<wire x1="670.56" y1="228.6" x2="662.94" y2="228.6" width="0.1524" layer="91"/>
+<label x="660.4" y="228.6" size="1.778" layer="95"/>
+</segment>
+</net>
+<net name="DBG3B" class="0">
+<segment>
+<pinref part="DBG3B" gate="G$1" pin="P$1"/>
+<wire x1="779.78" y1="58.42" x2="767.08" y2="58.42" width="0.1524" layer="91"/>
+<label x="767.08" y="58.42" size="1.778" layer="95"/>
+</segment>
+<segment>
+<pinref part="U7" gate="G$1" pin="PA3"/>
+<wire x1="670.56" y1="226.06" x2="662.94" y2="226.06" width="0.1524" layer="91"/>
+<label x="660.4" y="226.06" size="1.778" layer="95"/>
+</segment>
+</net>

Commit message: Switch the aux CAN to the LTC2875
Parts:
- U9: value TCAN334GSOT23 -> LTC2875; device pi3_hat:TCAN334GSOT23 -> pi3_hat:LTC2875; MF TI -> (none); MPN TCAN334GDCNT -> (none); POPULATE 1 -> (none)
Connections:
- new net CAN_SHDN: U7.PC6, U9.RS
- net GND: no longer U9.SHDN, U9.STB

Commit message: Flip rpi header start populating it, stop populating NRF header
Parts:
- J3: MF Wurth Elektornik -> (none); MPN 61300821121 -> (none); POPULATE 1 -> 0
- J4: device pinhead:PINHD-2X20 -> pi3_hat:PI3_HEADER2X20-FLIP; POPULATE 0 -> 1
Changed lines of the file:
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@@
 <part name="GND15" library="supply1" deviceset="GND" device=""/>
 <part name="GND16" library="supply1" deviceset="GND" device=""/>
-<part name="J4" library="pinhead" deviceset="PINHD-2X20" device="">
+<part name="J4" library="pi3_hat" deviceset="PI3_HEADER" device="2X20-FLIP">
 <attribute name="MF" value="Sullins"/>
 <attribute name="MPN" value="PPPC202LFBN-RC"/>
-<attribute name="POPULATE" value="0"/>
+<attribute name="POPULATE" value="1"/>
 </part>
 <part name="+3V6" library="supply1" deviceset="+3V3" device=""/>
@@
 <part name="+3V24" library="supply1" deviceset="+3V3" device=""/>
 <part name="J3" library="pinhead" deviceset="PINHD-2X4" device="">
-<attribute name="MF" value="Wurth Elektornik"/>
-<attribute name="MPN" value="61300821121"/>
-<attribute name="POPULATE" value="1"/>
+<attribute name="MF" value=""/>
+<attribute name="MPN" value=""/>
+<attribute name="POPULATE" value="0"/>
 </part>
 <part name="GND39" library="supply1" deviceset="GND" device=""/>

Commit message: Add IRQ lines to the rpi
Connections:
- new net AUX_IRQ1: J4.15, U7.PB0
- new net AUX_IRQ2: J4.16, U7.PB1
- new net AUX_IRQ3: J4.18, U7.PB2
- new net IFACEA_IRQ1: J4.37, U4.PB0
- new net IFACEB_IRQ1: J4.29, U11.PB0
Changed lines of the file:
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@@
+</segment>
+</net>
+<net name="AUX_IRQ1" class="0">
+<segment>
+<pinref part="U7" gate="G$1" pin="PB0"/>
+<wire x1="688.34" y1="205.74" x2="688.34" y2="187.96" width="0.1524" layer="91"/>
+<label x="688.34" y="187.96" size="1.778" layer="95" rot="R90"/>
+</segment>
+<segment>
+<pinref part="J4" gate="A" pin="15"/>
+<wire x1="53.34" y1="104.14" x2="30.48" y2="104.14" width="0.1524" layer="91"/>
+<label x="30.48" y="104.14" size="1.778" layer="95"/>
+</segment>
+</net>
+<net name="AUX_IRQ2" class="0">
+<segment>
+<pinref part="U7" gate="G$1" pin="PB1"/>
+<wire x1="690.88" y1="205.74" x2="690.88" y2="187.96" width="0.1524" layer="91"/>
+<label x="690.88" y="187.96" size="1.778" layer="95" rot="R90"/>
+</segment>
+<segment>
+<pinref part="J4" gate="A" pin="16"/>
+<wire x1="60.96" y1="104.14" x2="88.9" y2="104.14" width="0.1524" layer="91"/>
+<label x="83.82" y="104.14" size="1.778" layer="95"/>
+</segment>
+</net>
+<net name="AUX_IRQ3" class="0">
+<segment>
+<pinref part="U7" gate="G$1" pin="PB2"/>
+<wire x1="693.42" y1="205.74" x2="693.42" y2="187.96" width="0.1524" layer="91"/>
+<label x="693.42" y="187.96" size="1.778" layer="95" rot="R90"/>
+</segment>
+<segment>
+<pinref part="J4" gate="A" pin="18"/>
+<wire x1="60.96" y1="101.6" x2="88.9" y2="101.6" width="0.1524" layer="91"/>
+<label x="83.82" y="101.6" size="1.778" layer="95"/>
+</segment>
+</net>
+<net name="IFACEA_IRQ1" class="0">
+<segment>
+<pinref part="U4" gate="G$1" pin="PB0"/>
+<wire x1="375.92" y1="205.74" x2="375.92" y2="185.42" width="0.1524" layer="91"/>
+<label x="375.92" y="185.42" size="1.778" layer="95" rot="R90"/>
+</segment>
+<segment>
+<pinref part="J4" gate="A" pin="37"/>
+<wire x1="53.34" y1="76.2" x2="30.48" y2="76.2" width="0.1524" layer="91"/>
+<label x="30.48" y="76.2" size="1.778" layer="95"/>
+</segment>
+</net>
+<net name="IFACEB_IRQ1" class="0">
+<segment>
+<pinref part="J4" gate="A" pin="29"/>
+<wire x1="53.34" y1="86.36" x2="30.48" y2="86.36" width="0.1524" layer="91"/>
+<label x="30.48" y="86.36" size="1.778" layer="95"/>
+</segment>
+<segment>
+<pinref part="U11" gate="G$1" pin="PB0"/>
+<wire x1="373.38" y1="25.4" x2="373.38" y2="5.08" width="0.1524" layer="91"/>
+<label x="373.38" y="5.08" size="1.778" layer="95" rot="R90"/>
 </segment>
 </net>

Commit message: Expose debug pins on 0.1" headers, give 4 debug pins on the aux processor
Parts:
- removed DBG1A, DBG1B, DBG2A, DBG2B, DBG3A, DBG3B: PAD24AWG_PAD, pi3_hat:PAD24AWG_PAD
- added JP2: (no value), pinhead:PINHD-1X5
- added JP3, JP4: (no value), pinhead:PINHD-1X3
Connections:
- removed net DBG1A: DBG1A.P$1, U4.PB13
- removed net DBG1B: DBG1B.P$1, U4.PB12
- removed net DBG2A: DBG2A.P$1, U11.PB13
- removed net DBG2B: DBG2B.P$1, U11.PB12
- removed net DBG3A: DBG3A.P$1, U7.PA2
- removed net DBG3B: DBG3B.P$1, U7.PA3
- new net N$10: JP2.3, U7.PA2
- new net N$12: JP2.4, U7.PA1
- new net N$20: JP2.5, U7.PA0
- new net N$3: JP3.2, U11.PB12
- new net N$43: JP3.1, U11.PB13
- new net N$57: JP4.2, U4.PB12
- new net N$58: JP4.1, U4.PB13
- new net N$6: JP2.2, U7.PA3
- net GND: now also JP2.1, JP3.3, JP4.3
Other:
- moved on the sheet: C18
