File: hw/r4.5/pi3_hat.brd (EAGLE design)
At the start: 56.5 x 65 mm, 131 parts, among them J1 XT30P, J2 XT30P, U1 MAX17504ATP+T, U10 CAT24C32UDFN8, U11 STM32G474CEU6, U12 LTC2875, U13 LTC2875, U14 ICM-42688-P, U2 DMMT5401, U3 DMG2305UX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

Commit message: pi3hat r4.5
* Up voltage rating to 48V (technically 10V-54V)
* Replace CAN transceivers with 5V versions (with DNPs to support 3.3V
  ones if necessary)
* Use actual 120 ohm terminating resistors
* 0.1" I2C header
Parts:
- D12: device pi3_hat:SMF -> diode:DO214AA
Changed lines of the file:
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@@
 <element name="U9" library="pi3_hat" package="SOIC8" value="LTC2875" x="42.9" y="27.3" smashed="yes">
 <attribute name="MF" value="Analog" x="42.9" y="27.3" size="1.778" layer="27" display="off"/>
-<attribute name="MPN" value="TCAN1057AEVDRQ1" x="42.9" y="27.3" size="1.778" layer="27" display="off"/>
+<attribute name="MPN" value="TCAN1057AEVDRQ1‎" x="42.9" y="27.3" size="1.778" layer="27" display="off"/>
 <attribute name="NAME" x="42.3234" y="30.165" size="0.6" layer="25" font="vector" ratio="10" rot="SR0"/>
 <attribute name="POPULATE" value="1" x="42.9" y="27.3" size="1.778" layer="27" display="off"/>
@@
 <attribute name="VOLTAGE" value="" x="38.1" y="23.6" size="1.778" layer="27" display="off"/>
 </element>
-<element name="D12" library="pi3_hat" package="SMF" value="" x="31.2" y="1.5" smashed="yes">
+<element name="D12" library="diode" library_urn="urn:adsk.eagle:library:210" package="DO214AA" package3d_urn="urn:adsk.eagle:package:43433/2" value="" x="31.2" y="1.5" smashed="yes">
 <attribute name="MF" value="LITTLEFUSE" x="31.2" y="1.5" size="1.778" layer="27" display="off"/>
-<attribute name="MPN" value="SMF51A" x="31.2" y="1.5" size="1.778" layer="27" display="off"/>
-<attribute name="NAME" x="28.639" y="0.61" size="0.6" layer="25" ratio="10" rot="R90"/>
+<attribute name="MPN" value="SMBJ51A-13-F" x="31.2" y="1.5" size="1.778" layer="27" display="off"/>
+<attribute name="NAME" x="34.136" y="2.44" size="0.6" layer="25" ratio="10" rot="R270"/>
+<attribute name="POPULARITY" value="8" x="31.2" y="1.5" size="1.778" layer="27" display="off"/>
 <attribute name="POPULATE" value="1" x="31.2" y="1.5" size="1.778" layer="27" display="off"/>
-<attribute name="VALUE" value="" x="28.56" y="-1.206" size="1.27" layer="27" ratio="10"/>
+<attribute name="VALUE" x="28.56" y="-1.206" size="1.27" layer="27" ratio="10"/>
 </element>
 <element name="U5" library="pi3_hat" package="SOIC8" value="LTC2875" x="34.2" y="59.1" smashed="yes" rot="R270">
 <attribute name="MF" value="Analog" x="34.2" y="59.1" size="1.778" layer="27" rot="R270" display="off"/>
-<attribute name="MPN" value="TCAN1057AEVDRQ1" x="34.2" y="59.1" size="1.778" layer="27" rot="R270" display="off"/>
+<attribute name="MPN" value="TCAN1057AEVDRQ1‎" x="34.2" y="59.1" size="1.778" layer="27" rot="R270" display="off"/>
 <attribute name="NAME" x="36.7234" y="61.365" size="0.6" layer="25" ratio="10" rot="SR0"/>
 <attribute name="POPULATE" value="1" x="34.2" y="59.1" size="1.778" layer="27" rot="R270" display="off"/>
@@
 <element name="U6" library="pi3_hat" package="SOIC8" value="LTC2875" x="46.5" y="59.1" smashed="yes" rot="R270">
 <attribute name="MF" value="Analog" x="46.5" y="59.1" size="1.778" layer="27" rot="R270" display="off"/>
-<attribute name="MPN" value="TCAN1057AEVDRQ1" x="46.5" y="59.1" size="1.778" layer="27" rot="R270" display="off"/>
+<attribute name="MPN" value="TCAN1057AEVDRQ1‎" x="46.5" y="59.1" size="1.778" layer="27" rot="R270" display="off"/>
 <attribute name="NAME" x="48.9234" y="61.365" size="0.6" layer="25" ratio="10" rot="SR0"/>
 <attribute name="POPULATE" value="1" x="46.5" y="59.1" size="1.778" layer="27" rot="R270" display="off"/>
@@
 <element name="U12" library="pi3_hat" package="SOIC8" value="LTC2875" x="46.4" y="44.3" smashed="yes" rot="R270">
 <attribute name="MF" value="Analog" x="46.4" y="44.3" size="1.778" layer="27" rot="R270" display="off"/>
-<attribute name="MPN" value="TCAN1057AEVDRQ1" x="46.4" y="44.3" size="1.778" layer="27" rot="R270" display="off"/>
+<attribute name="MPN" value="TCAN1057AEVDRQ1‎" x="46.4" y="44.3" size="1.778" layer="27" rot="R270" display="off"/>
 <attribute name="NAME" x="49.0234" y="46.465" size="0.6" layer="25" ratio="10" rot="SR0"/>
 <attribute name="POPULATE" value="1" x="46.4" y="44.3" size="1.778" layer="27" rot="R270" display="off"/>
@@
 <element name="U13" library="pi3_hat" package="SOIC8" value="LTC2875" x="34.2" y="44.3" smashed="yes" rot="R270">
 <attribute name="MF" value="Analog" x="34.2" y="44.3" size="1.778" layer="27" rot="R270" display="off"/>
-<attribute name="MPN" value="TCAN1057AEVDRQ1" x="34.2" y="44.3" size="1.778" layer="27" rot="R270" display="off"/>
+<attribute name="MPN" value="TCAN1057AEVDRQ1‎" x="34.2" y="44.3" size="1.778" layer="27" rot="R270" display="off"/>
 <attribute name="NAME" x="31.335" y="43.5234" size="0.6" layer="25" ratio="10" rot="SR90"/>
 <attribute name="POPULATE" value="1" x="34.2" y="44.3" size="1.778" layer="27" rot="R270" display="off"/>
@@
 <via x="31.9" y="5.875" extent="1-16" drill="0.6"/>
 <via x="31.9" y="3.6" extent="1-16" drill="0.6"/>
-<via x="34.3" y="1.4" extent="1-16" drill="0.6"/>
+<via x="32.2" y="1.4" extent="1-16" drill="0.6"/>
 <polygon width="0.127" layer="1" isolate="0.7" thermals="no">
 <vertex x="32.4" y="8.7"/>
@@
 <vertex x="25.2" y="8.9"/>
 </polygon>
-<via x="34.3" y="2.6" extent="1-16" drill="0.6"/>
+<via x="31.9" y="2.5" extent="1-16" drill="0.6"/>
 <via x="31.9" y="4.725" extent="1-16" drill="0.6"/>
 </signal>
