File: hw/r4.5/pi3_hat.sch (EAGLE design)
At the start: 131 parts, among them J1 XT30P, J2 XT30P, U1 MAX17504ATP+T, U10 CAT24C32UDFN8, U11 STM32G474CEU6, U12 LTC2875, U13 LTC2875, U14 ICM-42688-P, U2 DMMT5401, U3 DMG2305UX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

Commit message: pi3hat r4.5
* Up voltage rating to 48V (technically 10V-54V)
* Replace CAN transceivers with 5V versions (with DNPs to support 3.3V
  ones if necessary)
* Use actual 120 ohm terminating resistors
* 0.1" I2C header
Parts:
- D12: value SMF -> (none); device pi3_hat:SMF -> diode:DIODE-DO214AA; MPN SMF51A -> SMBJ51A-13-F
- U12, U13, U5, U6, U9: MPN TCAN1057AEVDRQ1 -> TCAN1057AEVDRQ1‎
Other:
- moved on the sheet: D12
Changed lines of the file:
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@@
 <part name="U9" library="pi3_hat" deviceset="LTC2875" device="">
 <attribute name="MF" value="Analog"/>
-<attribute name="MPN" value="TCAN1057AEVDRQ1"/>
+<attribute name="MPN" value="TCAN1057AEVDRQ1‎"/>
 <attribute name="POPULATE" value="1"/>
 </part>
@@
 </part>
 <part name="GND63" library="supply1" deviceset="GND" device=""/>
-<part name="D12" library="pi3_hat" deviceset="SMF" device="" value="">
+<part name="D12" library="diode" library_urn="urn:adsk.eagle:library:210" deviceset="DIODE-" device="DO214AA" package3d_urn="urn:adsk.eagle:package:43433/2">
 <attribute name="MF" value="LITTLEFUSE"/>
-<attribute name="MPN" value="SMF51A"/>
+<attribute name="MPN" value="SMBJ51A-13-F"/>
 <attribute name="POPULATE" value="1"/>
 </part>
 <part name="U5" library="pi3_hat" deviceset="LTC2875" device="">
 <attribute name="MF" value="Analog"/>
-<attribute name="MPN" value="TCAN1057AEVDRQ1"/>
+<attribute name="MPN" value="TCAN1057AEVDRQ1‎"/>
 <attribute name="POPULATE" value="1"/>
 </part>
 <part name="U6" library="pi3_hat" deviceset="LTC2875" device="">
 <attribute name="MF" value="Analog"/>
-<attribute name="MPN" value="TCAN1057AEVDRQ1"/>
+<attribute name="MPN" value="TCAN1057AEVDRQ1‎"/>
 <attribute name="POPULATE" value="1"/>
 </part>
 <part name="U12" library="pi3_hat" deviceset="LTC2875" device="">
 <attribute name="MF" value="Analog"/>
-<attribute name="MPN" value="TCAN1057AEVDRQ1"/>
+<attribute name="MPN" value="TCAN1057AEVDRQ1‎"/>
 <attribute name="POPULATE" value="1"/>
 </part>
 <part name="U13" library="pi3_hat" deviceset="LTC2875" device="">
 <attribute name="MF" value="Analog"/>
-<attribute name="MPN" value="TCAN1057AEVDRQ1"/>
+<attribute name="MPN" value="TCAN1057AEVDRQ1‎"/>
 <attribute name="POPULATE" value="1"/>
 </part>
@@
 <pinref part="GND57" gate="1" pin="GND"/>
 <pinref part="D12" gate="G$1" pin="A"/>
-<wire x1="38.1" y1="259.08" x2="38.1" y2="251.46" width="0.1524" layer="91"/>
+<wire x1="38.1" y1="264.16" x2="38.1" y2="251.46" width="0.1524" layer="91"/>
 </segment>
 <segment>
@@
 <wire x1="48.26" y1="281.94" x2="48.26" y2="274.32" width="0.1524" layer="91"/>
 <junction x="48.26" y="281.94"/>
-<wire x1="38.1" y1="276.86" x2="38.1" y2="284.48" width="0.1524" layer="91"/>
+<wire x1="38.1" y1="269.24" x2="38.1" y2="284.48" width="0.1524" layer="91"/>
 <junction x="38.1" y="284.48"/>
 <label x="7.62" y="284.48" size="1.778" layer="95"/>
